File: eagle/MQTT_meteo_v2.0.brd (EAGLE design)
At the start: 77 x 45 mm, 35 parts, among them IC1 MCP9808-E/MS, J1 RJ-11, J2 RJ-11, U1 SPX3819M5-L-3-3/TR, U2 STM32F103C8T6-BREAKOUT, U3 ENC28J60-BREAKOUT, U4 BME280, U5 ESP8266-01S

Commit message: serial fix
Parts:
- moved JP2 55.0 mm to (73.4, 42.4)
- moved JP1 2.55 mm to (30.6, 2.67)
Connections:
- removed net ETH/ESP_RST: R9.1, U2.PA_3, U5.CH_PD
- removed net N$7: JP1.1, U5.TX
- removed net N$8: JP1.2, U5.RX
- removed net RXI: JP2.1, U2.PA_10
- removed net TXO: JP2.2, U2.PA_9
- new net RX_ESP: JP1.2, U2.PA_9, U5.RX
- new net RX_STM: JP2.2, U2.PA_3
- new net TX_ESP: JP1.1, U2.PA_10, U5.TX
- new net TX_STM: JP2.1, U2.PA_2
- net ENC/ESP_RST: now also R9.1, U2.PA_15, U5.CH_PD
Routing:
- net ETH/ESP_RST: track 55.0 -> 0.00 mm, vias 1 -> 0
- net RX_ESP: track 0.00 -> 45.7 mm
- net ENC/ESP_RST: track 0.00 -> 37.5 mm, vias 0 -> 1
- net TX_ESP: track 0.00 -> 36.6 mm
- net TXO: track 29.4 -> 0.00 mm
- net RXI: track 28.0 -> 0.00 mm
- net TX_STM: track 0.00 -> 27.3 mm
- net RX_STM: track 0.00 -> 23.2 mm
- net N$8: track 16.1 -> 0.00 mm
- net N$7: track 7.40 -> 0.00 mm
Other:
- outline, holes or cut-outs redrawn
- board text added: "IO0"
- board text removed: "GPIO0"
- board text removed: "RX_STM"
- board text removed: "TX_STM"
