File: eagle/MQTT_meteo_v2.0.sch (EAGLE design)
At the start: 35 parts, among them IC1 MCP9808-E/MS, J1 RJ-11, J2 RJ-11, U1 SPX3819M5-L-3-3/TR, U2 STM32F103C8T6-BREAKOUT, U3 ENC28J60-BREAKOUT, U4 BME280, U5 ESP8266-01S

Commit message: serial fix
Connections:
- removed net ETH/ESP_RST: R9.1, U2.PA_3, U5.CH_PD
- removed net N$7: JP1.1, U5.TX
- removed net N$8: JP1.2, U5.RX
- removed net RXI: JP2.1, U2.PA_10
- removed net TXO: JP2.2, U2.PA_9
- new net RX_ESP: JP1.2, U2.PA_9, U5.RX
- new net RX_STM: JP2.2, U2.PA_3
- new net TX_ESP: JP1.1, U2.PA_10, U5.TX
- new net TX_STM: JP2.1, U2.PA_2
- net ENC/ESP_RST: now also R9.1, U2.PA_15, U5.CH_PD
Other:
- moved on the sheet: JP1, JP2
